Commit message: Moteus working version with JTC

File: proxima_description/robots/moteus_motor.xacro (robot description, xacro)
@@ -50,4 +50,5 @@
       <axis xyz="0 0 1"/>
       <dynamics damping="0.0" friction="0.0"/>
+      <limit lower="-1.5" upper="1.5" effort="100.0" velocity="1.0"/>
     </joint>
     <link name="${name}_output">
